Commit message: fix collision bug

File: source/b2_z1/b2_z1/assets/b2_z1/b2_z1.urdf (robot description, URDF)
Before this commit: robot b2_description, 46 links, 45 joints
Links:
- removed link dummy_target
- removed link link_gun
- removed link link_mounter
- link FL_calf: geometry collision box size=0.02 0.028 0.035; collision box size=0.05 0.0245 0.018
- link FL_hip_rotor: geometry 
- link FL_thigh: geometry collision box size=0.25 0.028 0.04; visual mesh filename=b2_description/meshes/FL_thigh.dae
- link FR_calf: geometry collision box size=0.02 0.028 0.035; collision box size=0.05 0.0245 0.018
- link FR_hip_rotor: geometry 
- link RL_calf: geometry collision box size=0.02 0.028 0.035; collision box size=0.05 0.0245 0.018
- link RL_hip_rotor: geometry 
- link RR_calf: geometry collision box size=0.02 0.028 0.035; collision box size=0.05 0.0245 0.018
- link RR_hip_rotor: geometry 
- link base_link: geometry collision box size=0.5 0.28 0.15; visual mesh filename=b2_description/meshes/base_link_wo_lidar.obj
- link link00: geometry visual mesh filename=z1_description/meshes/visual/z1_Link00.dae
- link link04: geometry visual mesh filename=z1_description/meshes/visual/z1_Link04.dae
Joints:
- removed joint joint_gun_mounter
- removed joint joint_mounter
- removed joint link_dummy_target_joint
- joint joint0: axis 0 0 1 -> (none); limit lower=-2.6179939 upper=2.6179939 effort=30 velocity=3.1415 -> (none)

Commit message: base training

File: source/b2_z1/b2_z1/assets/b2_z1/b2_z1.urdf (robot description, URDF)
Before this commit: robot b2_description, 43 links, 42 joints
Links:
- added link dummy_target, mass 0
Joints:
- added joint link_dummy_target_joint: type fixed, parent link06, child dummy_target, origin xyz=0.1 0 0 rpy=0 0 0, axis 1 0 0
