Commit message: init train

File: source/b2_z1/b2_z1/assets/b2_z1/b2_z1_gun.urdf (robot description, URDF)
Before this commit: robot b2_description, 46 links, 45 joints
Links:
- link link_gun: geometry collision cylinder length=1.1 radius=0.028; visual mesh filename=gun/meshes/gun_base_shifted_center.stl
Joints:
- joint joint0: origin xyz=0 0 0.09 rpy=0 0 0 -> xyz=0 0 0.09 rpy=0 0 1.5708
- joint joint_gun_mounter: origin xyz=0.0 0 0.05 rpy=-1.5708 0 1.5708 -> xyz=0.0 0 0.05 rpy=0 0 1.5708
- joint link_dummy_target_joint: origin xyz=0.0 0.21 -0.6 rpy=-3.14159 1.0472 1.5708 -> xyz=0.0 -0.03 -0.62 rpy=-3.14159 1.5708 1.5708

Commit message: vis traj

File: source/b2_z1/b2_z1/assets/b2_z1/b2_z1_gun.urdf (robot description, URDF)
Before this commit: robot b2_description, 46 links, 45 joints
Joints:
- joint joint_gun_mounter: origin xyz=0.0 0 0.05 rpy=0 0 1.5708 -> xyz=0.0 0 -0.2 rpy=0 0 1.5708
