Commit message: ee_drived vel tracking  init

File: source/b2_z1/b2_z1/assets/b2_z1/b2_z1_gun.urdf (robot description, URDF)
Before this commit: robot b2_description, 46 links, 45 joints
Joints:
- joint joint0: origin xyz=0 0 0.09 rpy=0 0 1.5708 -> xyz=0 0 0.09 rpy=0 0 0

Commit message: feat: add rear-facing arm visual trajectory control

File: source/b2_z1/b2_z1/assets/b2_z1/b2_z1_gun.urdf (robot description, URDF)
Before this commit: robot b2_description, 46 links, 45 joints
Joints:
- joint joint0: origin xyz=0 0 0.09 rpy=0 0 0 -> xyz=0 0 0.09 rpy=0 0 3.14159265

File: source/b2_z1/b2_z1/assets/b2_z1/b2_z1_no_stick.urdf (robot description, URDF)
Before this commit: robot b2_description, 46 links, 45 joints
Joints:
- joint joint0: origin xyz=0 0 0.09 rpy=0 0 0 -> xyz=0 0 0.09 rpy=0 0 3.14159265
